File: Archivos Kicad/Termometro.sch (KiCad schematic (older format))
At the start: 24 parts, among them SW1 SW_Push, SW2 SW_Push, SW3 SW_Push, SW4 SW_Push, U1 LM358, U2 CC56-12EWA

Commit message: Docs-Datasheet/microentrenador-2021-v1.pdf
Parts:
- D1: symbol Diode:1N4148 -> Termometro-rescue:1N4148-Diode
- H1, H2, H3, H4: symbol Mechanical:MountingHole -> Termometro-rescue:MountingHole-Mechanical
- R1, R10, R11, R12, R2, R3, R4, R5, R6, R7, R8, R9: symbol Device:R -> Termometro-rescue:R-Device
- SW1, SW2, SW3, SW4: symbol Switch:SW_Push -> Termometro-rescue:SW_Push-Switch
- U1: symbol Amplifier_Operational:LM358 -> Termometro-rescue:LM358-Amplifier_Operational
- U2: symbol Display_Character:CA56-12CGKWA -> Termometro-rescue:CA56-12CGKWA-Display_Character
Changed lines of the file:
@@
 CC4
 $Comp
-L Device:R R5
+L Termometro-rescue:R-Device R5
 U 1 1 5D22AFBA
 P 8100 3450
@@
 $EndComp
 $Comp
-L Device:R R4
+L Termometro-rescue:R-Device R4
 U 1 1 5D22B012
 P 7750 3550
@@
 $EndComp
 $Comp
-L Device:R R6
+L Termometro-rescue:R-Device R6
 U 1 1 5D22B057
 P 8100 3650
@@
 	8500 4250 8450 4300
 $Comp
-L Display_Character:CA56-12CGKWA U2
+L Termometro-rescue:CA56-12CGKWA-Display_Character U2
 U 1 1 5D2241E2
 P 6300 3250
@@
 a
 $Comp
-L Device:R R1
+L Termometro-rescue:R-Device R1
 U 1 1 5D22EF7C
 P 4050 3250
@@
 	3750 3250 3900 3250
 $Comp
-L power:GND #PWR0102
+L Termometro-rescue:GND-power #PWR0102
 U 1 1 5D2343A5
 P 3300 4950
@@
 $EndComp
 $Comp
-L power:+5V #PWR0107
+L Termometro-rescue:+5V-power #PWR0107
 U 1 1 5D236852
 P 3950 4300
@@
 Wire Wire Line
 	3950 4300 4050 4300
-Connection ~ 3950 4300
 Wire Wire Line
 	3750 3250 3750 3750
 $Comp
-L power:GND #PWR0106
+L Termometro-rescue:GND-power #PWR0106
 U 1 1 5D23682F
 P 4350 4750
@@
 Connection ~ 4350 4300
 $Comp
-L Device:R R7
+L Termometro-rescue:R-Device R7
 U 1 1 5D2366ED
 P 4200 4300
@@
 	4550 3650 4350 3650
 $Comp
-L power:GND #PWR0101
+L Termometro-rescue:GND-power #PWR0101
 U 1 1 5D22F037
 P 4550 4050
@@
 Connection ~ 4550 3650
 $Comp
-L Device:R R2
+L Termometro-rescue:R-Device R2
 U 1 1 5D22EFCE
 P 4550 3800
@@
 	3300 4950 3300 4700
 $Comp
-L power:+5V #PWR0104
+L Termometro-rescue:+5V-power #PWR0104
 U 1 1 5D236589
 P 3400 2650
@@
 DPX
 $Comp
-L Diode:1N4148 D1
+L Termometro-rescue:1N4148-Diode D1
 U 1 1 5D236798
 P 4350 4600
@@
 Connection ~ 3750 3750
 $Comp
-L Amplifier_Operational:LM358 U1
+L Termometro-rescue:LM358-Amplifier_Operational U1
 U 1 1 5D22A72A
 P 4050 3750
@@
 	5750 5350 5750 5300
 $Comp
-L power:GND #PWR0112
+L Termometro-rescue:GND-power #PWR0112
 U 1 1 5D23D4A7
 P 5750 5650
@@
 $EndComp
 $Comp
-L Device:R R9
+L Termometro-rescue:R-Device R9
 U 1 1 5D23C8DF
 P 5750 5500
@@
 $EndComp
 $Comp
-L Device:R R12
+L Termometro-rescue:R-Device R12
 U 1 1 5D23C8A1
 P 7550 5150
@@
 $EndComp
 $Comp
-L Device:R R11
+L Termometro-rescue:R-Device R11
 U 1 1 5D23C818
 P 6950 5150
@@
 $EndComp
 $Comp
-L Device:R R10
+L Termometro-rescue:R-Device R10
 U 1 1 5D23C7D8
 P 6350 5150
@@
 $EndComp
 $Comp
-L Device:R R8
+L Termometro-rescue:R-Device R8
 U 1 1 5D23C6F7
 P 5750 5150
@@
 $EndComp
 $Comp
-L power:+5V #PWR0111
+L Termometro-rescue:+5V-power #PWR0111
 U 1 1 5D23C672
 P 7550 4600
@@
 $EndComp
 $Comp
-L power:+5V #PWR0110
+L Termometro-rescue:+5V-power #PWR0110
 U 1 1 5D23C647
 P 6950 4600
@@
 $EndComp
 $Comp
-L power:+5V #PWR0109
+L Termometro-rescue:+5V-power #PWR0109
 U 1 1 5D23C61C
 P 6350 4600
@@
 $EndComp
 $Comp
-L power:+5V #PWR0108
+L Termometro-rescue:+5V-power #PWR0108
 U 1 1 5D23C5F1
 P 5750 4600
@@
 $EndComp
 $Comp
-L Switch:SW_Push SW4
+L Termometro-rescue:SW_Push-Switch SW4
 U 1 1 5D23C5B3
 P 7550 4800
@@
 $EndComp
 $Comp
-L Switch:SW_Push SW3
+L Termometro-rescue:SW_Push-Switch SW3
 U 1 1 5D23C573
 P 6950 4800
@@
 $EndComp
 $Comp
-L Switch:SW_Push SW2
+L Termometro-rescue:SW_Push-Switch SW2
 U 1 1 5D23C533
 P 6350 4800
@@
 $EndComp
 $Comp
-L Switch:SW_Push SW1
+L Termometro-rescue:SW_Push-Switch SW1
 U 1 1 5D23C3F9
 P 5750 4800
@@
 $EndComp
 $Comp
-L power:+5V #PWR0105
+L Termometro-rescue:+5V-power #PWR0105
 U 1 1 5D2365AF
 P 5200 5050
@@
 $EndComp
 $Comp
-L power:GND #PWR0103
+L Termometro-rescue:GND-power #PWR0103
 U 1 1 5D235035
 P 5200 5650
@@
 $EndComp
 $Comp
-L Amplifier_Operational:LM358 U1
+L Termometro-rescue:LM358-Amplifier_Operational U1
 U 3 1 5D234FC0
 P 5300 5350
@@
 $EndComp
 $Comp
-L power:PWR_FLAG #FLG0101
+L Termometro-rescue:PWR_FLAG-power #FLG0101
 U 1 1 613D8A7F
 P 2550 5850
@@
 $EndComp
 $Comp
-L power:GND #PWR0113
+L Termometro-rescue:GND-power #PWR0113
 U 1 1 613D8A85
 P 2550 5950
@@
 	3300 4700 3300 4650
 $Comp
-L Mechanical:MountingHole H3
+L Termometro-rescue:MountingHole-Mechanical H3
 U 1 1 61412614
 P 4050 5800
@@
 $EndComp
 $Comp
-L Mechanical:MountingHole H1
+L Termometro-rescue:MountingHole-Mechanical H1
 U 1 1 61409849
 P 3150 5800
@@
 $EndComp
 $Comp
-L Mechanical:MountingHole H2
+L Termometro-rescue:MountingHole-Mechanical H2
 U 1 1 6142C6E0
 P 3150 6100
@@
 $EndComp
 $Comp
-L Mechanical:MountingHole H4
+L Termometro-rescue:MountingHole-Mechanical H4
 U 1 1 6142F660
 P 4050 6100
@@
 $EndComp
 $Comp
-L Device:R R3
+L Termometro-rescue:R-Device R3
 U 1 1 5D22AF4D
 P 7750 3350
@@
 Wire Wire Line
 	2700 3250 2300 3250
-Wire Bus Line
-	8500 3450 8500 4250
-Wire Bus Line
-	2200 2430 2200 5200
-Wire Bus Line
-	4750 2750 4750 5200
 Text Label 2300 3250 0    50   ~ 0
 CC3
+Wire Bus Line
+	8500 3450 8500 4250
+Wire Bus Line
+	2200 2430 2200 5200
+Wire Bus Line
+	4750 2750 4750 5200
 $EndSCHEMATC
