File: Archivos Kicad/Termometro.kicad_pcb (KiCad board)
At the start: 2 copper layers, 53.3 x 66 mm, 24 parts, among them SW1 SW_Push, SW2 SW_Push, SW3 SW_Push, SW4 SW_Push, U1 LM358, U2 CC56-12EWA

Commit message: Docs-Datasheet/microentrenador-2021-v1.pdf
Routing:
- net GND: track 101.3 -> 103.1 mm
- net +5V: track 103.6 -> 104.2 mm

Commit message: modified:   Archivos Kicad/Termometro.kicad_pcb  Untracked files: 	Archivos FREECad/desktop.ini 	Archivos Kicad/LibreriaCustumLemos.pretty/desktop.ini 	Archivos Kicad/Termometro-backups/ 	Archivos Kicad/Termometro.kicad_prl 	Archivos Kicad/Termometro.kicad_pro 	Archivos Kicad/Termometro.kicad_sch 	Archivos Kicad/_autosave-Termometro.sch 	Archivos Kicad/desktop.ini 	Archivos Kicad/footprint_display/desktop.ini 	Archivos Simulacion/desktop.ini 	Docs-Datasheet/desktop.ini 	desktop.ini 	programaDemo/desktop.ini
Parts:
- removed H1, H2: MountingHole, MountingHole:MountingHole_3.2mm_M3
- moved R4 27.3 mm to (119.4, 94.2), turned to 90 degrees
- moved R2 21.9 mm to (136.7, 126.5)
- moved R3 20.6 mm to (144.8, 101.2), turned to 0 degrees
- moved R5 19.4 mm to (142.4, 93.3), turned to 0 degrees
- moved R6 18.4 mm to (144.7, 106.0), turned to 0 degrees
- moved R9 10.6 mm to (116.9, 127.5), turned to 90 degrees
- moved H4 6.73 mm to (115.3, 76.4)
- moved H3 5.33 mm to (158.5, 76.4)
Connections:
- A1 pad 1: /CC4 -> unconnected-(A1-Pad1)
- A1 pad 10: /e -> /d
- A1 pad 11: /f -> /e
- A1 pad 12: /a -> /f
- A1 pad 13: /CC1 -> /g
- A1 pad 14: /CC2 -> /DPX
- A1 pad 15: Net-(A1-Pad15) -> /CC3
- A1 pad 16: Net-(A1-Pad16) -> /CC4
- A1 pad 17: Net-(A1-Pad17) -> unconnected-(A1-Pad17)
- A1 pad 18: Net-(A1-Pad18) -> unconnected-(A1-Pad18)
- A1 pad 2: /b -> unconnected-(A1-Pad2)
- A1 pad 21: Net-(A1-Pad21) -> unconnected-(A1-Pad21)
- A1 pad 22: Net-(A1-Pad22) -> unconnected-(A1-Pad22)
- A1 pad 23: Net-(A1-Pad23) -> unconnected-(A1-Pad23)
- A1 pad 24: Net-(A1-Pad24) -> unconnected-(A1-Pad24)
- A1 pad 25: Net-(A1-Pad25) -> unconnected-(A1-Pad25)
- A1 pad 26: Net-(A1-Pad26) -> unconnected-(A1-Pad26)
- A1 pad 28: Net-(A1-Pad28) -> unconnected-(A1-Pad28)
- A1 pad 3: Net-(A1-Pad3) -> unconnected-(A1-Pad3)
- A1 pad 30: Net-(A1-Pad30) -> unconnected-(A1-Pad30)
- A1 pad 5: /CC3 -> /CC1
- A1 pad 6: /g -> /CC2
- A1 pad 7: /c -> /a
- A1 pad 8: /DPX -> /b
- A1 pad 9: /d -> /c
Routing:
- net GND: track 103.1 -> 24.7 mm
- net /a: track 25.1 -> 66.8 mm
- net Net-(R6-Pad2): track 8.09 -> 44.3 mm, vias 0 -> 2
- net /CC4: track 6.81 -> 30.4 mm
- net Net-(R4-Pad2): track 46.4 -> 25.1 mm
- net /g: track 10.2 -> 31.4 mm, vias 0 -> 2
- net Net-(R3-Pad2): track 33.7 -> 54.2 mm
- net +5V: track 104.2 -> 117.9 mm, vias 2 -> 0
- net /DPX: track 10.7 -> 23.2 mm
- net /A0: track 26.7 -> 17.3 mm
- net Net-(R5-Pad2): track 38.9 -> 29.6 mm
- net Net-(R1-Pad1): track 27.1 -> 18.7 mm
- net /b: track 23.5 -> 27.7 mm
- net /f: track 26.2 -> 28.8 mm, vias 0 -> 2
- net /CC3: track 5.78 -> 3.50 mm
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Other:
- board size 53.3 x 66 mm -> 53.3 x 67.8 mm
- net class Default removed
- net class Power removed
- board text removed: "TERMÓMETRO"

Commit message: correccion del board
Routing:
- net GND: track 24.7 -> 98.6 mm
- removed copper zone on B.Cu, net GND
Changed lines of the file:
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@@
   (segment (start 136.673165 116.343767) (end 140.082165 116.343767) (width 1) (layer "B.Cu") (net 1))
   (segment (start 142.283665 120.156267) (end 140.102165 117.974767) (width 1) (layer "B.Cu") (net 1))
+  (segment (start 159.204186 110.926788) (end 157.782165 109.504767) (width 1) (layer "B.Cu") (net 2))
+  (segment (start 116.861165 125.625767) (end 118.057165 124.429767) (width 1) (layer "B.Cu") (net 2))
+  (segment (start 154.382165 109.579767) (end 152.484665 107.682267) (width 1) (layer "B.Cu") (net 2))
+  (segment (start 152.484665 107.682267) (end 152.484665 107.557267) (width 1) (layer "B.Cu") (net 2))
+  (segment (start 147.404665 97.718267) (end 147.404665 102.477267) (width 1) (layer "B.Cu") (net 2))
+  (segment (start 118.057165 124.429767) (end 134.782165 124.429767) (width 1) (layer "B.Cu") (net 2))
+  (segment (start 154.457165 109.504767) (end 154.382165 109.579767) (width 1) (layer "B.Cu") (net 2))
+  (segment (start 157.782165 109.504767) (end 154.457165 109.504767) (width 1) (layer "B.Cu") (net 2))
+  (segment (start 155.024665 124.451767) (end 157.160165 124.451767) (width 1) (layer "B.Cu") (net 2))
+  (segment (start 155.088165 131.690767) (end 155.571165 131.690767) (width 1) (layer "B.Cu") (net 2))
   (segment (start 154.961165 131.817767) (end 154.961165 135.754767) (width 1) (layer "B.Cu") (net 2))
+  (segment (start 159.204186 122.407746) (end 159.204186 110.926788) (width 1) (layer "B.Cu") (net 2))
   (segment (start 139.049548 128.88015) (end 152.277548 128.88015) (width 1) (layer "B.Cu") (net 2))
+  (segment (start 135.057165 124.704767) (end 135.057165 124.887767) (width 1) (layer "B.Cu") (net 2))
   (segment (start 136.673165 126.503767) (end 139.049548 128.88015) (width 1) (layer "B.Cu") (net 2))
+  (segment (start 157.507165 124.798767) (end 157.160165 124.451767) (width 1) (layer "B.Cu") (net 2))
+  (segment (start 147.404665 102.477267) (end 152.484665 107.557267) (width 1) (layer "B.Cu") (net 2))
+  (segment (start 157.507165 129.754767) (end 157.507165 124.798767) (width 1) (layer "B.Cu") (net 2))
+  (segment (start 116.861165 127.519767) (end 116.861165 125.625767) (width 1) (layer "B.Cu") (net 2))
   (segment (start 155.088165 131.690767) (end 154.961165 131.817767) (width 1) (layer "B.Cu") (net 2))
+  (segment (start 157.160165 124.451767) (end 159.204186 122.407746) (width 1) (layer "B.Cu") (net 2))
+  (segment (start 135.057165 124.887767) (end 136.673165 126.503767) (width 1) (layer "B.Cu") (net 2))
+  (segment (start 155.571165 131.690767) (end 157.507165 129.754767) (width 1) (layer "B.Cu") (net 2))
   (segment (start 152.277548 128.88015) (end 155.088165 131.690767) (width 1) (layer "B.Cu") (net 2))
+  (segment (start 134.782165 124.429767) (end 135.057165 124.704767) (width 1) (layer "B.Cu") (net 2))
+  (segment (start 152.484665 107.557267) (end 152.484665 112.958267) (width 1) (layer "B.Cu") (net 2))
   (segment (start 154.941165 101.210767) (end 157.374165 101.210767) (width 1) (layer "B.Cu") (net 3))
   (segment (start 159.787165 98.797767) (end 159.787165 88.041139) (width 1) (layer "B.Cu") (net 3))
@@
   (segment (start 116.861165 117.359767) (end 120.244765 117.359767) (width 1) (layer "B.Cu") (net 38))
   (segment (start 117.242165 117.339767) (end 117.242165 117.212767) (width 1) (layer "B.Cu") (net 38))
-  (zone (net 2) (net_name "GND") (layer "B.Cu") (hatch edge 0.508)
-    (connect_pads (clearance 1.5))
-    (min_thickness 0.254) (filled_areas_thickness no)
-    (fill yes (thermal_gap 0.5) (thermal_bridge_width 0.5) (smoothing chamfer) (radius 0.7))
-    (polygon
-      (pts
-        (xy 162.962165 143.374767)
-        (xy 110.892165 143.374767)
-        (xy 110.892165 73.524767)
-        (xy 162.962165 73.524767)
-      )
-    )
-  )
 )
